File: src/botCode/PCB/PacBot_2021-2022.kicad_pcb (KiCad board)
At the start: 2 copper layers, 127 x 76.2 mm, 24 parts, among them J1 conn_imu, J2 conn_motor-encoder_L, J3 conn_motor-encoder_R, J4 RPi_GPIO, J5 Conn_Batt, U1 L7805, U2 Teensy-LC, U3 VL6180X, U4 DRV8835, U5 VL6180X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

Commit message: updated pcb
Parts:
- moved C7 6.69 mm to (120.4, 98.6)
- moved U1 5.36 mm to (167.2, 127.5), turned to 0 degrees
- moved C2 2.28 mm to (170.8, 124.9), turned to 180 degrees
- moved J5 2.11 mm to (168.6, 135.5), turned to 0 degrees
Routing:
- net +5V: track 0.00 -> 105.7 mm
- net /VBAT: track 0.00 -> 71.2 mm
- net GND: track 0.00 -> 2.75 mm
Changed lines of the file:
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@@
   )
   (footprint "Connector_JST:JST_PH_B2B-PH-K_1x02_P2.00mm_Vertical" (layer "F.Cu")
-    (at 170.63 135.08 180)
+    (at 168.56 135.48)
     (descr "JST PH series connector, B2B-PH-K (http://www.jst-mfg.com/product/pdf/eng/ePH.pdf), generated with kicad-footprint-generator")
     (tags "connector JST PH side entry")
@@
     (fp_line (start -1.11 -2.11) (end -2.36 -2.11) (layer "F.Fab") (width 0.1))
     (fp_line (start 3.95 -1.7) (end -1.95 -1.7) (layer "F.Fab") (width 0.1))
-    (pad "1" thru_hole roundrect (at 0 0 180) (size 1.2 1.75) (drill 0.75) (layers *.Cu *.Mask) (roundrect_rratio 0.208333)
+    (pad "1" thru_hole roundrect (at 0 0) (size 1.2 1.75) (drill 0.75) (layers *.Cu *.Mask) (roundrect_rratio 0.208333)
       (net 48 "/VBAT") (pinfunction "Pin_1") (pintype "passive"))
-    (pad "2" thru_hole oval (at 2 0 180) (size 1.2 1.75) (drill 0.75) (layers *.Cu *.Mask)
+    (pad "2" thru_hole oval (at 2 0) (size 1.2 1.75) (drill 0.75) (layers *.Cu *.Mask)
       (net 2 "GND") (pinfunction "Pin_2") (pintype "passive"))
     (model "${KICAD6_3DMODEL_DIR}/Connector_JST.3dshapes/JST_PH_B2B-PH-K_1x02_P2.00mm_Vertical.wrl"
@@
   )
   (footprint "Capacitor_SMD:C_0603_1608Metric" (layer "F.Cu")
-    (at 168.67 124.08)
+    (at 170.79 124.93 180)
     (descr "Capacitor SMD 0603 (1608 Metric), square (rectangular) end terminal, IPC_7351 nominal, (Body size source: IPC-SM-782 page 76, https://www.pcb-3d.com/wordpress/wp-content/uploads/ipc-sm-782a_amendment_1_and_2.pdf), generated with kicad-footprint-generator")
     (tags "capacitor")
@@
     (property "Sheetname" "")
     (attr smd)
-    (fp_text reference "C2" (at 0 -1.43) (layer "F.SilkS")
+    (fp_text reference "C2" (at -2.57 0.07) (layer "F.SilkS")
       (effects (font (size 1 1) (thickness 0.15)))
     )
@@
     (fp_line (start 0.8 -0.4) (end 0.8 0.4) (layer "F.Fab") (width 0.1))
     (fp_line (start -0.8 0.4) (end -0.8 -0.4) (layer "F.Fab") (width 0.1))
-    (pad "1" smd roundrect (at -0.775 0) (size 0.9 0.95) (layers "F.Cu" "F.Paste" "F.Mask") (roundrect_rratio 0.25)
+    (pad "1" smd roundrect (at -0.775 0 180) (size 0.9 0.95) (layers "F.Cu" "F.Paste" "F.Mask") (roundrect_rratio 0.25)
       (net 3 "+5V") (pintype "passive"))
-    (pad "2" smd roundrect (at 0.775 0) (size 0.9 0.95) (layers "F.Cu" "F.Paste" "F.Mask") (roundrect_rratio 0.25)
+    (pad "2" smd roundrect (at 0.775 0 180) (size 0.9 0.95) (layers "F.Cu" "F.Paste" "F.Mask") (roundrect_rratio 0.25)
       (net 2 "GND") (pintype "passive"))
     (model "${KICAD6_3DMODEL_DIR}/Capacitor_SMD.3dshapes/C_0603_1608Metric.wrl"
@@
   )
   (footprint "Connector_Stocko:Stocko_MKS_1653-6-0-303_1x3_P2.50mm_Vertical" (layer "F.Cu")
-    (at 172.55 127.03 180)
+    (at 167.21 127.51)
     (descr "Stocko MKS 16xx series connector, (https://www.stocko-contact.com/downloads/steckverbindersystem-raster-2,5-mm.pdf#page=15), generated with kicad-footprint-generator")
     (tags "Stocko RFK MKS 16xx")
@@
     (fp_arc (start -3.6 -3.25) (mid -3.453553 -3.603553) (end -3.1 -3.75) (layer "F.Fab") (width 0.1))
     (fp_arc (start -3.1 3.75) (mid -3.453553 3.603553) (end -3.6 3.25) (layer "F.Fab") (width 0.1))
-    (pad "1" thru_hole roundrect (at 0 0 180) (size 1.5 2) (drill 1) (layers *.Cu *.Mask) (roundrect_rratio 0.25)
+    (pad "1" thru_hole roundrect (at 0 0) (size 1.5 2) (drill 1) (layers *.Cu *.Mask) (roundrect_rratio 0.25)
       (net 48 "/VBAT") (pinfunction "IN") (pintype "power_in"))
-    (pad "2" thru_hole oval (at 2.5 0 180) (size 1.5 2) (drill 1) (layers *.Cu *.Mask)
+    (pad "2" thru_hole oval (at 2.5 0) (size 1.5 2) (drill 1) (layers *.Cu *.Mask)
       (net 2 "GND") (pinfunction "GND") (pintype "power_in"))
-    (pad "3" thru_hole oval (at 5 0 180) (size 1.5 2) (drill 1) (layers *.Cu *.Mask)
+    (pad "3" thru_hole oval (at 5 0) (size 1.5 2) (drill 1) (layers *.Cu *.Mask)
       (net 3 "+5V") (pinfunction "OUT") (pintype "power_out"))
     (model "${KICAD6_3DMODEL_DIR}/Connector_Stocko.3dshapes/Stocko_MKS_1653-6-0-303_1x3_P2.50mm_Vertical.wrl"
@@
   )
   (footprint "Capacitor_SMD:C_0603_1608Metric" (layer "B.Cu")
-    (at 127.11 98.72 90)
+    (at 120.42 98.57 90)
     (descr "Capacitor SMD 0603 (1608 Metric), square (rectangular) end terminal, IPC_7351 nominal, (Body size source: IPC-SM-782 page 76, https://www.pcb-3d.com/wordpress/wp-content/uploads/ipc-sm-782a_amendment_1_and_2.pdf), generated with kicad-footprint-generator")
     (tags "capacitor")
@@
   (via (at 159.63 69.93) (size 2.5) (drill 2.2) (layers "F.Cu" "B.Cu") (net 0))
   (via (at 134.63 71.18) (size 2.5) (drill 2.2) (layers "F.Cu" "B.Cu") (net 0))
+  (segment (start 169.71 127.51) (end 169.71 125.235) (width 1) (layer "F.Cu") (net 2))
+  (segment (start 169.71 125.235) (end 170.015 124.93) (width 1) (layer "F.Cu") (net 2))
+  (segment (start 170.63 135.08) (end 170.61 135.06) (width 0.25) (layer "F.Cu") (net 2))
+  (segment (start 170.63 135.08) (end 170.62 135.07) (width 0.25) (layer "F.Cu") (net 2))
+  (segment (start 172.21 125.575) (end 171.565 124.93) (width 1) (layer "F.Cu") (net 3))
+  (segment (start 172.21 127.51) (end 172.21 125.575) (width 1) (layer "F.Cu") (net 3))
+  (segment (start 147.4 123.69) (end 143.56 119.85) (width 1) (layer "B.Cu") (net 3))
+  (segment (start 119.07 82.07) (end 117.875 80.875) (width 1) (layer "B.Cu") (net 3))
+  (segment (start 170.21 123.69) (end 167.16 123.69) (width 1) (layer "B.Cu") (net 3))
+  (segment (start 122.79 93.62) (end 121.88 92.71) (width 1) (layer "B.Cu") (net 3))
+  (segment (start 172.21 127.51) (end 172.21 125.69) (width 1) (layer "B.Cu") (net 3))
+  (segment (start 121.87 82.05) (end 121.85 82.07) (width 1) (layer "B.Cu") (net 3))
+  (segment (start 121.85 82.07) (end 119.07 82.07) (width 1) (layer "B.Cu") (net 3))
+  (segment (start 172.21 125.69) (end 170.21 123.69) (width 1) (layer "B.Cu") (net 3))
+  (segment (start 143.56 119.85) (end 143.56 96.44) (width 1) (layer "B.Cu") (net 3))
+  (segment (start 166.26 123.69) (end 167.16 123.69) (width 1) (layer "B.Cu") (net 3))
+  (segment (start 143.56 96.44) (end 140.74 93.62) (width 1) (layer "B.Cu") (net 3))
+  (segment (start 121.88 82.05) (end 121.87 82.05) (width 1) (layer "B.Cu") (net 3))
+  (segment (start 121.88 92.71) (end 121.88 82.05) (width 1) (layer "B.Cu") (net 3))
+  (segment (start 140.74 93.62) (end 122.79 93.62) (width 1) (layer "B.Cu") (net 3))
+  (segment (start 117.875 83.415) (end 119.07 82.22) (width 1) (layer "B.Cu") (net 3))
+  (segment (start 119.07 82.22) (end 119.07 82.07) (width 1) (layer "B.Cu") (net 3))
+  (segment (start 167.16 123.69) (end 147.4 123.69) (width 1) (layer "B.Cu") (net 3))
+  (segment (start 162.43 119.86) (end 166.26 123.69) (width 1) (layer "B.Cu") (net 3))
   (via (at 127.63 69.93) (size 2.5) (drill 2.2) (layers "F.Cu" "B.Cu") (net 15))
   (via (at 99.63 98.299) (size 2.5) (drill 2.2) (layers "F.Cu" "B.Cu") (net 38))
+  (segment (start 127.25 114.71) (end 127.25 101.73) (width 1.5) (layer "B.Cu") (net 48))
+  (segment (start 129.03 99.95) (end 130.9 99.95) (width 1.5) (layer "B.Cu") (net 48))
+  (segment (start 167.21 134.13) (end 167.21 127.51) (width 2) (layer "B.Cu") (net 48))
+  (segment (start 167.21 127.51) (end 140.05 127.51) (width 1.5) (layer "B.Cu") (net 48))
+  (segment (start 127.25 101.73) (end 129.03 99.95) (width 1.5) (layer "B.Cu") (net 48))
+  (segment (start 140.05 127.51) (end 127.25 114.71) (width 1.5) (layer "B.Cu") (net 48))
+  (segment (start 168.56 135.48) (end 167.21 134.13) (width 2) (layer "B.Cu") (net 48))
   (via (at 187.63 98.299) (size 2.5) (drill 2.2) (layers "F.Cu" "B.Cu") (net 50))
   (via (at 187.63 111.761) (size 2.5) (drill 2.2) (layers "F.Cu" "B.Cu") (net 54))
   (via (at 99.63 111.761) (size 2.5) (drill 2.2) (layers "F.Cu" "B.Cu") (net 78))
-  (group "" (id 788cf3b5-a2c6-4528-899a-4918adb8d527)
-    (members
-      24b72b0d-63b8-4e06-89d0-e94dcf39a600
-      4e677390-a246-4ca0-954c-746e0870f88f
-    )
-  )
 )

Commit message: working on PCB
Parts:
- C7: moved to F.Cu
- moved J2 42.0 mm to (127.1, 131.0)
- moved J3 42.0 mm to (127.1, 89.0)
- moved C7 15.3 mm to (128.7, 111.5), turned to -90 degrees
- moved C5 1.00 mm to (111.3, 87.6)
- moved J4 1.00 mm to (115.6, 105.0)
- turned U4 to 180 degrees
Routing:
- net Net-(J3-Pad5): track 0.00 -> 28.1 mm
- net Net-(J3-Pad6): track 0.00 -> 27.4 mm
- net Net-(J2-Pad5): track 0.00 -> 19.6 mm
- net Net-(J2-Pad6): track 0.00 -> 19.5 mm
- net /VBAT: track 71.2 -> 84.6 mm
- net +5V: track 105.7 -> 117.4 mm

Commit message: update kicad
Parts:
- C1, C10, C3, C4, C5, C6, C8, C9: moved to F.Cu
- moved C9 103.6 mm to (92.4, 108.8), turned to 90 degrees
- moved C10 83.8 mm to (105.6, 130.8)
- moved C5 70.9 mm to (181.7, 79.3), turned to 0 degrees
- moved C7 63.7 mm to (189.4, 130.9), turned to 180 degrees
- moved C8 46.1 mm to (97.9, 79.2), turned to 0 degrees
- moved C4 44.5 mm to (128.3, 111.3), turned to -90 degrees
- moved C1 43.9 mm to (137.1, 101.4), turned to -90 degrees
- moved C6 35.3 mm to (110.8, 78.9), turned to 180 degrees
- moved C3 25.9 mm to (194.8, 101.3), turned to 90 degrees
Connections:
- U3 pad 6: /IRA_EN -> /IRB_EN
- U5 pad 6: /IRB_EN -> /IRE_EN
- U8 pad 6: /IRE_EN -> /IRA_EN
Routing:
- net /SDA0: track 0.00 -> 393.2 mm
- net /SCL0: track 0.00 -> 390.9 mm
- net +3V3: track 0.00 -> 99.0 mm, vias 0 -> 28
- net /IRE_EN: track 0.00 -> 96.9 mm, vias 1 -> 0
- net /IRB_EN: track 0.00 -> 90.3 mm
- net /COM_TO_TN: track 0.00 -> 89.7 mm
- net /COM_TO_PI: track 0.00 -> 82.9 mm
- net /IRC_EN: track 0.00 -> 67.7 mm
- net /L_EN_A: track 0.00 -> 57.8 mm
- net /L_EN_B: track 0.00 -> 57.5 mm
- net /R_EN_B: track 0.00 -> 37.4 mm
- net /R_EN_A: track 0.00 -> 37.1 mm
- net /SDA1: track 0.00 -> 36.8 mm
- net /IRF_EN: track 0.00 -> 35.7 mm
- net /SCL1: track 0.00 -> 34.2 mm
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- added copper zone on F.Cu, net +3V3
- added copper zone on B.Cu, net GND
