File: src/botCode/PCB/PacBot_2021-2022.kicad_pcb (KiCad board)
At the start: 2 copper layers, 127 x 76.2 mm, 24 parts, among them J1 conn_imu, J2 conn_motor-encoder_L, J3 conn_motor-encoder_R, J4 RPi_GPIO, J5 Conn_Batt, U1 L7805, U2 Teensy-LC, U3 VL6180X, U4 DRV8835, U5 VL6180X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

Commit message: updated PCB
Parts:
- J1, U3, U5, U6, U7, U8, U9: moved to B.Cu
- moved C3 7.74 mm to (195.3, 109.0), turned to -90 degrees
- moved C5 7.68 mm to (189.4, 79.4), turned to 180 degrees
- moved C8 7.62 mm to (105.5, 79.5), turned to 180 degrees
- moved C9 7.51 mm to (92.7, 101.3), turned to -90 degrees
- moved C10 7.49 mm to (98.1, 130.5), turned to 0 degrees
- moved C7 7.48 mm to (181.9, 130.5), turned to 0 degrees
- moved C1 7.28 mm to (137.0, 108.7), turned to 90 degrees
Routing:
- net +3V3: track 99.0 -> 117.6 mm, vias 28 -> 32
- net /IMU_PS0: track 25.9 -> 39.5 mm
- net /IRC_EN: track 67.7 -> 80.1 mm
- net /IRE_EN: track 96.9 -> 84.8 mm
- net /IRB_EN: track 90.3 -> 100.5 mm
- net /IMU_PS1: track 25.9 -> 35.7 mm
- net /IMU_INT: track 25.9 -> 32.4 mm
- net /SDA1: track 36.8 -> 31.2 mm
- net /SCL0: track 390.9 -> 396.0 mm
- net /IRA_EN: track 19.7 -> 24.7 mm
- net /IMU_RST: track 29.4 -> 33.5 mm
- net /IRF_EN: track 35.7 -> 31.7 mm
- net /IRD_EN: track 16.5 -> 20.4 mm
- net /SCL1: track 34.2 -> 31.7 mm
- net /IMU_ADR: track 25.9 -> 27.6 mm
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