File: src/botCode/PCB/PacBot_2021-2022.kicad_sch (KiCad schematic)
At the start: 24 parts, among them J1 conn_imu, J2 conn_motor-encoder_L, J3 conn_motor-encoder_R, J4 RPi_GPIO, J5 Conn_Batt, U1 L7805, U2 Teensy-LC, U3 VL6180X, U4 DRV8835, U5 VL6180X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

Commit message: schematic updated
Connections:
- net IRA_EN: now also U8.6 (GPIO0); no longer U3.6 (GPIO0)
- net IRB_EN: now also U3.6 (GPIO0); no longer U5.6 (GPIO0)
- net IRE_EN: now also U5.6 (GPIO0); no longer U8.6 (GPIO0)
Changed lines of the file:
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@@
     (effects (font (size 1.27 1.27)) (justify right bottom))
   )
-  (label "IRB_EN" (at 270.51 140.97 180)
+  (label "IRE_EN" (at 270.51 140.97 180)
     (effects (font (size 1.27 1.27)) (justify right bottom))
   )
@@
     (effects (font (size 1.27 1.27)) (justify left bottom))
   )
-  (label "IRE_EN" (at 270.51 213.36 180)
+  (label "IRA_EN" (at 270.51 213.36 180)
     (effects (font (size 1.27 1.27)) (justify right bottom))
   )
@@
     (effects (font (size 1.27 1.27)) (justify left bottom))
   )
-  (label "IRA_EN" (at 270.51 116.84 180)
+  (label "IRB_EN" (at 270.51 116.84 180)
     (effects (font (size 1.27 1.27)) (justify right bottom))
   )
